Commit message: Update robot.urdf.xacro

File: bringup/description/robot.urdf.xacro (robot description, xacro)
@@ -1,12 +1,22 @@
-// NEEDS TO BE CHANGED AS PER OWN PARAMETERS
 <?xml version="1.0"?>
-<robot xmlns:xacro="http://ros.org/wiki/xacro" name="omni_robot">
-  <!-- Include parts -->
-  <xacro:include filename="$(find motor_controller)/urdf/base.xacro"/>
-  <xacro:include filename="$(find motor_controller)/urdf/wheels.xacro"/>
-  <xacro:include filename="$(find motor_controller)/urdf/control.xacro"/>
-  <!-- Instantiate -->
-  <xacro:base/>
-  <xacro:wheels/>
-  <xacro:control/>
+<robot xmlns:xacro="http://ros.org/wiki/xacro">
+  <xacro:macro name="pi" params="3.1415926535897931" />
+  <material name="gray">
+    <color rgba="0.8 0.8 0.8 1.0"/>
+  </material>
+  <material name="black">
+    <color rgba="0 0 0 1.0"/>
+  </material>
+  <material name="white">
+    <color rgba="1.0 1.0 1.0 1.0"/>
+  </material>
+  <material name="red">
+    <color rgba="1.0 0 0 1.0"/>
+  </material>
+  <material name="light_red">
+    <color rgba="1.0 0.5 0.5 1.0"/>
+  </material>
+  <material name="yellow">
+    <color rgba="0 1.0 1.0 1.0"/>
+  </material>
 </robot>
